File: schematic/a277d-led-tachometer.kicad_pcb (KiCad board)
At the start: 2 copper layers, 140 x 60 mm, 61 parts, among them IC1 A277D, J1 Terminal Block, J2 Terminal Block, J3 DC-005 Power Jack, J4 Conn_01x02_Pin, J5 Conn_01x02_Pin, P1 100K, P2 100K, P3 100K, T1 BC547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

Commit message: Footprints updated
Parts:
- C3, C5, C6: footprint Capacitor_THT:CP_Radial_D6.3mm_P2.50mm -> Capacitor_THT:CP_Radial_D5.0mm_P2.00mm
- C4: footprint Capacitor_THT:CP_Radial_D6.3mm_P2.50mm -> Capacitor_THT:CP_Radial_D13.0mm_P5.00mm
- moved T2 5.14 mm to (50.7, 35.9)
- moved C2 3.50 mm to (49.5, 29.5)
- moved Z2 2.50 mm to (59.0, 31.4)
- moved T1 2.14 mm to (50.7, 23.9)
- moved C4 1.12 mm to (50.0, 50.0)
- moved C3 1.00 mm to (40.0, 50.0)
- moved Z1 1.00 mm to (59.0, 17.9)
Routing:
- net Net-(IC1-VCC): track 108.4 -> 113.2 mm
- net Net-(Z1-K): track 40.3 -> 37.6 mm
- net Net-(T2-B): track 7.38 -> 9.59 mm
- net Net-(T2-C): track 36.0 -> 34.1 mm
- net +12V: track 223.2 -> 224.9 mm
- net Net-(T1-B): track 30.1 -> 28.8 mm
- net Net-(T1-C): track 37.4 -> 36.4 mm
