File: schematic/a277d-led-tachometer.kicad_sch (KiCad schematic)
At the start: 52 parts, among them IC1 A277D, J1 Terminal Block, J2 Terminal Block, J3 DC-005 Power Jack, J4 Conn_01x02_Pin, J5 Conn_01x02_Pin, P1 100K, P2 100K, P3 100K, T1 BC547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

Commit message: Footprints updated
Parts:
- C3, C5, C6: footprint Capacitor_THT:CP_Radial_D6.3mm_P2.50mm -> Capacitor_THT:CP_Radial_D5.0mm_P2.00mm
- C4: footprint Capacitor_THT:CP_Radial_D6.3mm_P2.50mm -> Capacitor_THT:CP_Radial_D13.0mm_P5.00mm
- IC1: footprint Package_DIP:DIP-18_W7.62mm -> Package_DIP:DIP-18_W7.62mm_Socket
Changed lines of the file:
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@@
       (effects (font (size 1.27 1.27)) (justify left))
     )
-    (property "Footprint" "Capacitor_THT:CP_Radial_D6.3mm_P2.50mm" (at 172.4152 149.86 0)
+    (property "Footprint" "Capacitor_THT:CP_Radial_D5.0mm_P2.00mm" (at 172.4152 149.86 0)
       (effects (font (size 1.27 1.27)) hide)
     )
@@
       (effects (font (size 1.27 1.27)) (justify left))
     )
-    (property "Footprint" "Capacitor_THT:CP_Radial_D6.3mm_P2.50mm" (at 121.6152 104.14 0)
+    (property "Footprint" "Capacitor_THT:CP_Radial_D5.0mm_P2.00mm" (at 121.6152 104.14 0)
       (effects (font (size 1.27 1.27)) hide)
     )
@@
       (effects (font (size 1.27 1.27)) (justify left))
     )
-    (property "Footprint" "Capacitor_THT:CP_Radial_D6.3mm_P2.50mm" (at 223.2152 149.86 0)
+    (property "Footprint" "Capacitor_THT:CP_Radial_D5.0mm_P2.00mm" (at 223.2152 149.86 0)
       (effects (font (size 1.27 1.27)) hide)
     )
@@
       (effects (font (size 1.27 1.27)))
     )
-    (property "Footprint" "Package_DIP:DIP-18_W7.62mm" (at 210.82 -27.61 0)
+    (property "Footprint" "Package_DIP:DIP-18_W7.62mm_Socket" (at 210.82 -27.61 0)
       (effects (font (size 1.27 1.27)) (justify left top) hide)
     )
@@
       (effects (font (size 1.27 1.27)) (justify left))
     )
-    (property "Footprint" "Capacitor_THT:CP_Radial_D6.3mm_P2.50mm" (at 164.7952 104.14 0)
-      (effects (font (size 1.27 1.27)) hide)
-    )
+    (property "Footprint" "Capacitor_THT:CP_Radial_D13.0mm_P5.00mm" (at 164.7952 104.14 0)
+      (effects (font (size 1.27 1.27)) hide)
+    )

Commit message: 12V Power LED resistor updated on schematic
Parts:
- R11: value 1k -> 2k
Changed lines of the file:
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@@
       (effects (font (size 1.27 1.27)) (justify left))
     )
-    (property "Value" "1k" (at 266.7 139.7 0)
+    (property "Value" "2k" (at 266.7 139.7 0)
       (effects (font (size 1.27 1.27)) (justify left))
     )
